File: Radio/Radio.kicad_pcb (KiCad board)
At the start: 2 copper layers, 116 x 128 mm, 61 parts, among them J1 Conn_01x06_Pin, J2 Conn_01x02_Pin, J3 Conn_01x01_Pin, J4 Conn_Coaxial, J5 Conn_01x01_Pin, J6 Conn_01x02_Pin, J7 Conn_01x04_Pin, J8 Conn_01x14_Pin, J9 Conn_01x14_Pin, Q1 BC547, Q2 BC547, Q3 BC547, SW1 SW_Push, SW2 SW_Push, SW3 SW_Push, SW4 SW_Push, SW5 SW_Push, SW6 SW_Push, SW8 RotaryEncoder_Switch, U1 L7805, U2 LM386, U3 Aux_flush, U4 TL072, U5 Switch, U6 Aux_flush, U7 Aux_flush, U8 Aux_flush, Y1 Crystal

Commit message: Add files via upload
Parts:
- removed the ? at (114.4, 96.9)
- removed the ? at (72.9, 96.9)
- removed the ? at (114.4, 81.4)
- removed the ? at (72.9, 112.4)
- removed the ? at (114.4, 112.4)
- removed U5: Switch, Library:Switch
- added C11: C, Capacitor_THT:C_Rect_L9.0mm_W2.5mm_P7.50mm_MKT, F.Cu at (136.9, 66.9)
- added C12: C, Capacitor_THT:C_Rect_L9.0mm_W2.5mm_P7.50mm_MKT, F.Cu at (130.7, 110.4)
- added C13: C, Capacitor_THT:C_Rect_L7.2mm_W2.5mm_P5.00mm_FKS2_FKP2_MKS2_MKP2, F.Cu at (93.4, 47.2)
- added J10: Conn_01x02_Pin, Connector_PinHeader_2.54mm:PinHeader_1x03_P2.54mm_Vertical, F.Cu at (126.7, 67.9)
- added SW7: SW_SPDT, Connector_PinHeader_2.54mm:PinHeader_1x03_P2.54mm_Vertical, F.Cu at (165.3, 68.7)
- J9: footprint Connector_PinHeader_2.54mm:PinHeader_1x14_P2.54mm_Vertical -> Connector_PinSocket_2.54mm:PinSocket_1x14_P2.54mm_Vertical
Connections:
- J7 pad 1: +3V3 -> GND
- J7 pad 2: GND -> +3V3
- U9 pad 10: +3V3 -> Net-(J10-Pin_2)
Routing:
- net +3V3: track 167.3 -> 193.8 mm
- net Net-(J10-Pin_2): track 0.00 -> 12.6 mm
- net Net-(SW7-C): track 17.1 -> 12.0 mm
- net ANT: track 67.0 -> 68.3 mm
