File: Radio/Radio.kicad_sch (KiCad schematic)
At the start: 51 parts, among them J1 Conn_01x06_Pin, J2 Conn_01x02_Pin, J3 Conn_01x01_Pin, J4 Conn_Coaxial, J5 Conn_01x01_Pin, J6 Conn_01x02_Pin, J7 Conn_01x04_Pin, J8 Conn_01x14_Pin, J9 Conn_01x14_Pin, Q1 BC547, Q2 BC547, Q3 BC547, SW1 SW_Push, SW2 SW_Push, SW3 SW_Push, SW4 SW_Push, SW5 SW_Push, SW6 SW_Push, SW7 SW_SPDT, SW8 RotaryEncoder_Switch, U1 L7805, U2 LM386, U3 Aux_flush, U4 TL072, U6 Aux_flush, U7 Aux_flush, U8 Aux_flush, Y1 Crystal

Commit message: Add files via upload
Parts:
- added C11, C12: C, Capacitor_THT:C_Rect_L9.0mm_W2.5mm_P7.50mm_MKT, symbol Device:C
- added C13: C, Capacitor_THT:C_Rect_L7.2mm_W2.5mm_P5.00mm_FKS2_FKP2_MKS2_MKP2, symbol Device:C
- added J10: Conn_01x02_Pin, Connector_PinHeader_2.54mm:PinHeader_1x03_P2.54mm_Vertical, symbol Connector:Conn_01x03_Pin
- Q1, Q2, Q3: footprint Package_TO_SOT_THT:TO-92_Inline -> Package_TO_SOT_THT:TO-92_Inline_Wide
- SW7: footprint (none) -> Connector_PinHeader_2.54mm:PinHeader_1x03_P2.54mm_Vertical
Connections:
- net +3V3: now also J7.2 (Pin_2), C11.1, C12.1, C13.1, J10.3 (Pin_3); no longer J7.1 (Pin_1), U9.10 (SENB)
- net GND: now also J7.1 (Pin_1), C11.2, C12.2, C13.2, J10.1 (Pin_1); no longer J7.2 (Pin_2)
- new net: J10.2 (Pin_2), U9.10 (SENB)
